Commit message: Refactoring camera names

File: kulbu_description/urdf/kulbu.xacro (robot description, xacro)
@@ -42,17 +42,17 @@
     </link>
     <!-- EffortJointInterface/VelocityJointInterface -->
-    <wheel fb="front" lr="left"  tX="1" tY="1"  mu="0.3" interface="VelocityJointInterface" />
-    <wheel fb="front" lr="right" tX="1" tY="-1" mu="0.3" interface="VelocityJointInterface" />
-    <wheel fb="back" lr="left"  tX="-1" tY="1"  mu="0.3" interface="VelocityJointInterface" />
-    <wheel fb="back" lr="right" tX="-1" tY="-1" mu="0.3" interface="VelocityJointInterface" />
-    <wheel fb="mid" lr="left"  tX="0" tY="1"  mu="0.3" interface="VelocityJointInterface" />
-    <wheel fb="mid" lr="right" tX="0" tY="-1" mu="0.3" interface="VelocityJointInterface" />
-    <joint name="camera_joint" type="fixed">
-        <axis xyz="0 1 0" />
-        <origin xyz="${chassisLength/2} 0 ${chassisHeight+0.05}" rpy="0 0 0"/> <!-- ${PI/2} -->
-        <parent link="chassis_link"/>
-        <child link="camera_link"/>
-    </joint>
-    <link name="camera_link">
+    <wheel fb="front" lr="left"  tX="1"  tY="1"   mu="0.3" interface="VelocityJointInterface" />
+    <wheel fb="front" lr="right" tX="1"  tY="-1"  mu="0.3" interface="VelocityJointInterface" />
+    <wheel fb="back"  lr="left"  tX="-1" tY="1"   mu="0.3" interface="VelocityJointInterface" />
+    <wheel fb="back"  lr="right" tX="-1" tY="-1"  mu="0.3" interface="VelocityJointInterface" />
+    <wheel fb="mid"   lr="left"  tX="0"  tY="1"   mu="0.3" interface="VelocityJointInterface" />
+    <wheel fb="mid"   lr="right" tX="0"  tY="-1"  mu="0.3" interface="VelocityJointInterface" />
+    <joint name="camera_depth_joint" type="fixed">
+        <axis xyz="0 1 0" />
+        <origin xyz="${chassisLength/2} 0 ${chassisHeight+0.05}" rpy="0 0 0"/> <!-- Rotate sideways: ${PI/2} -->
+        <parent link="chassis_link"/>
+        <child link="camera_depth_link"/>
+    </joint>
+    <link name="camera_depth_link">
         <collision>
             <origin xyz="0 0 0" rpy="0 0 0"/>
@@ -75,11 +75,11 @@
     </link>
     <!-- OpenNI coordinates are different, transform for display in rvis -->
-    <joint name="camera_optical_joint" type="fixed">
-        <axis xyz="0 1 0" />
-        <origin xyz="${cameraSize/2} ${(cameraSize*3)/2} ${cameraSize/2}" rpy="${PI/2} ${PI} ${PI/2}"/>
-        <parent link="camera_link"/>
-        <child link="camera_optical_link"/>
-    </joint>
-    <link name="camera_optical_link">
+    <joint name="camera_depth_optical_joint" type="fixed">
+        <axis xyz="0 1 0" />
+        <origin xyz="${cameraSize/2} 0 ${cameraSize/2}" rpy="${PI/2} ${PI} ${PI/2}"/>
+        <parent link="camera_depth_link"/>
+        <child link="camera_depth_optical_link"/>
+    </joint>
+    <link name="camera_depth_optical_link">
         <collision>
             <origin xyz="0 0 0" rpy="0 0 0"/>
@@ -182,5 +182,5 @@
     <joint name="laser_joint" type="fixed">
         <axis xyz="0 1 0" />
-        <origin xyz="${chassisLength/2} 0 ${chassisHeight+0.1}" rpy="0 0 0"/><!-- ${PI/2} -->
+        <origin xyz="${chassisLength/2} 0 ${chassisHeight+0.2}" rpy="0 0 0"/><!-- ${PI/2} -->
         <parent link="chassis_link"/>
         <child link="laser_link"/>

File: kulbu_description/urdf/materials.xacro (robot description, xacro)
@@ -9,4 +9,7 @@
     <material name="green">
       <color rgba="0.0 0.8 0.0 1.0"/>
+    </material>
+    <material name="yellow">
+      <color rgba="0.8 0.8 0.2 1.0"/>
     </material>
     <material name="grey">

Commit message: Sonar range sensor

File: kulbu_description/urdf/kulbu.xacro (robot description, xacro)
@@ -206,4 +206,16 @@
         </inertial>
     </link>
+    <!-- Range
+    0.130899694 = 7.5deg (middle comes to here)
+    0.261799388 = 15deg (2nd centre here)
+    0.392699082 = 22.5deg (2nd comes to here)
+    0.523598776 = 30deg (3rd centre here)
+    0.654498469 = 37.5deg
+    -->
+    <sensor_range name="range_0"  linX="${0.02+chassisLength/2}" linY="0"     linZ="${chassisHeight}" angR="0" angP="0" angY="0" />
+    <sensor_range name="range_1l" linX="${0.02+chassisLength/2}" linY="0.05"  linZ="${chassisHeight}" angR="0" angP="0" angY="0.261799388" />
+    <sensor_range name="range_2l" linX="${0.02+chassisLength/2}" linY="0.10"  linZ="${chassisHeight}" angR="0" angP="0" angY="0.523598776" />
+    <sensor_range name="range_1r" linX="${0.02+chassisLength/2}" linY="-0.05" linZ="${chassisHeight}" angR="0" angP="0" angY="-0.261799388" />
+    <sensor_range name="range_2r" linX="${0.02+chassisLength/2}" linY="-0.10" linZ="${chassisHeight}" angR="0" angP="0" angY="-0.523598776" />
     <!-- IMU -->
     <joint name="imu_joint" type="fixed">

File: kulbu_description/urdf/macros.xacro (robot description, xacro)
@@ -2,40 +2,40 @@
 <robot name="kulbu" xmlns:xacro="http://www.ros.org/wiki/xacro">
     <macro name="cylinder_inertia" params="m r h">
-      <inertia  ixx="${m*(3*r*r+h*h)/12}" ixy = "0" ixz = "0"
-        iyy="${m*(3*r*r+h*h)/12}" iyz = "0"
-        izz="${m*r*r/2}"
-      />
+        <inertia  ixx="${m*(3*r*r+h*h)/12}" ixy="0" ixz="0"
+          iyy="${m*(3*r*r+h*h)/12}" iyz="0"
+          izz="${m*r*r/2}"
+        />
     </macro>
     <macro name="box_inertia" params="m x y z">
-      <inertia  ixx="${m*(y*y+z*z)/12}" ixy = "0" ixz = "0"
-        iyy="${m*(x*x+z*z)/12}" iyz = "0"
-        izz="${m*(x*x+z*z)/12}"
-      />
+        <inertia  ixx="${m*(y*y+z*z)/12}" ixy="0" ixz="0"
+          iyy="${m*(x*x+z*z)/12}" iyz="0"
+          izz="${m*(x*x+z*z)/12}"
+        />
     </macro>
     <macro name="sphere_inertia" params="m r">
-      <inertia  ixx="${2*m*r*r/5}" ixy = "0" ixz = "0"
-        iyy="${2*m*r*r/5}" iyz = "0"
-        izz="${2*m*r*r/5}"
-      />
+        <inertia  ixx="${2*m*r*r/5}" ixy="0" ixz="0"
+          iyy="${2*m*r*r/5}" iyz="0"
+          izz="${2*m*r*r/5}"
+        />
     </macro>
     <macro name="wheel" params="fb lr tX tY mu interface">
         <link name="${fb}_${lr}_wheel">
           <collision>
-            <origin xyz="0 0 0" rpy="0 ${PI/2} ${PI/2}" />
-            <geometry>
-              <cylinder length="${wheelWidth}" radius="${wheelRadius}"/>
-            </geometry>
+              <origin xyz="0 0 0" rpy="0 ${PI/2} ${PI/2}" />
+              <geometry>
+                  <cylinder length="${wheelWidth}" radius="${wheelRadius}"/>
+              </geometry>
           </collision>
           <visual>
-            <origin xyz="0 0 0" rpy="0 ${PI/2} ${PI/2}" />
-            <geometry>
-              <cylinder length="${wheelWidth}" radius="${wheelRadius}"/>
-            </geometry>
-            <material name="black"/>
+              <origin xyz="0 0 0" rpy="0 ${PI/2} ${PI/2}" />
+              <geometry>
+                  <cylinder length="${wheelWidth}" radius="${wheelRadius}"/>
+              </geometry>
+              <material name="black"/>
           </visual>
           <inertial>
-            <origin xyz="0 0 0" rpy="0 ${PI/2} ${PI/2}" />
-            <mass value="${wheelMass}"/>
-            <cylinder_inertia m="${wheelMass}" r="${wheelRadius}" h="${wheelWidth}"/>
+              <origin xyz="0 0 0" rpy="0 ${PI/2} ${PI/2}" />
+              <mass value="${wheelMass}"/>
+              <cylinder_inertia m="${wheelMass}" r="${wheelRadius}" h="${wheelWidth}"/>
           </inertial>
         </link>
@@ -66,3 +66,61 @@
         </transmission>
     </macro>
+    <macro name="sensor_range" params="name linX linY linZ angR angP angY">
+        <joint name="range_${name}_joint" type="fixed">
+            <axis xyz="0 1 0" />
+            <origin xyz="${linX} ${linY} ${linZ}" rpy="${angR} ${angP} ${angY}" />
+            <parent link="chassis_link" />
+            <child link="range_${name}_link" />
+        </joint>
+        <link name="range_${name}_link">
+            <collision>
+                <origin xyz="0 0 0" rpy="0 0 0" />
+                <geometry>
+                    <box size="0.0 0.0 0.0" />
+                </geometry>
+            </collision>
+            <visual>
+                <origin xyz="0 0 0" rpy="0 0 0" />
+                <geometry>
+                    <box size="0.015 0.045 0.02" />
+                </geometry>
+                <material name="blue" />
+            </visual>
+            <inertial>
+                <mass value="0.001" />
+                <origin xyz="0 0 0" rpy="0 0 0" />
+                <inertia ixx="0.000000017" ixy="0" ixz="0" iyy="0.000000017" iyz="0" izz="0.000000017" />
+            </inertial>
+        </link>
+        <gazebo reference="range_${name}_link">
+            <material>Gazebo/Blue</material>
+            <sensor type="ray" name="range_${name}">
+                <update_rate>10</update_rate>
+                <ray>
+                    <range>
+                        <min>0.02</min>
+                        <max>4.00</max>
+                        <resolution>0.01</resolution>
+                    </range>
+                    <scan>
+                        <horizontal>
+                            <samples>1</samples>
+                            <min_angle>-0.130899694</min_angle>
+                            <max_angle>0.130899694</max_angle>
+                        </horizontal>
+                        <vertical>
+                            <samples>1</samples>
+                            <min_angle>-0.130899694</min_angle>
+                            <max_angle>0.130899694</max_angle>
+                        </vertical>
+                    </scan>
+                </ray>
+                <plugin name="gazebo_ros_sonar_${name}_controller" filename="libhector_gazebo_ros_sonar.so">
+                    <gaussianNoise>0.000</gaussianNoise>
+                    <topicName>$(arg ns)/${name}</topicName>
+                    <frameId>range_${name}_link</frameId>
+                </plugin>
+            </sensor>
+        </gazebo>
+    </macro>
 </robot>

Commit message: Attempts at contact sensor

File: kulbu_description/urdf/kulbu.xacro (robot description, xacro)
@@ -212,10 +212,15 @@
     0.523598776 = 30deg (3rd centre here)
     0.654498469 = 37.5deg
+    0.785398163 = 45deg
     -->
-    <sensor_range name="range_0"  linX="${0.02+chassisLength/2}" linY="0"     linZ="${chassisHeight}" angR="0" angP="0" angY="0" />
-    <sensor_range name="range_1l" linX="${0.02+chassisLength/2}" linY="0.05"  linZ="${chassisHeight}" angR="0" angP="0" angY="0.261799388" />
-    <sensor_range name="range_2l" linX="${0.02+chassisLength/2}" linY="0.10"  linZ="${chassisHeight}" angR="0" angP="0" angY="0.523598776" />
-    <sensor_range name="range_1r" linX="${0.02+chassisLength/2}" linY="-0.05" linZ="${chassisHeight}" angR="0" angP="0" angY="-0.261799388" />
-    <sensor_range name="range_2r" linX="${0.02+chassisLength/2}" linY="-0.10" linZ="${chassisHeight}" angR="0" angP="0" angY="-0.523598776" />
+    <sensor_range name="range_0"  linX="${0.02+chassisLength/2}" linY="0"     linZ="${chassisHeight+0.3}" angR="0" angP="0" angY="0" />
+    <sensor_range name="range_1l" linX="${0.02+chassisLength/2}" linY="0.05"  linZ="${chassisHeight+0.3}" angR="0" angP="0" angY="0.261799388" />
+    <sensor_range name="range_2l" linX="${0.02+chassisLength/2}" linY="0.10"  linZ="${chassisHeight+0.3}" angR="0" angP="0" angY="0.523598776" />
+    <sensor_range name="range_3l" linX="${0.02+chassisLength/2}" linY="0.15"  linZ="${chassisHeight+0.3}" angR="0" angP="0" angY="0.785398163" />
+    <sensor_range name="range_1r" linX="${0.02+chassisLength/2}" linY="-0.05" linZ="${chassisHeight+0.3}" angR="0" angP="0" angY="-0.261799388" />
+    <sensor_range name="range_2r" linX="${0.02+chassisLength/2}" linY="-0.10" linZ="${chassisHeight+0.3}" angR="0" angP="0" angY="-0.523598776" />
+    <sensor_range name="range_3r" linX="${0.02+chassisLength/2}" linY="-0.15" linZ="${chassisHeight+0.3}" angR="0" angP="0" angY="-0.785398163" />
+    <!--sensor_bump name="bump_l" linX="${chassisLength/2}" linY="0.15"  linZ="${chassisHeight}" angR="0" angP="0" angY="0.785398163" /-->
+    <!--sensor_bump name="bump_r" linX="${chassisLength/2}" linY="-0.15" linZ="${chassisHeight}" angR="0" angP="0" angY="-0.785398163" /-->
     <!-- IMU -->
     <joint name="imu_joint" type="fixed">

File: kulbu_description/urdf/macros.xacro (robot description, xacro)
@@ -67,11 +67,11 @@
     </macro>
     <macro name="sensor_range" params="name linX linY linZ angR angP angY">
-        <joint name="range_${name}_joint" type="fixed">
+        <joint name="${name}_joint" type="fixed">
             <axis xyz="0 1 0" />
             <origin xyz="${linX} ${linY} ${linZ}" rpy="${angR} ${angP} ${angY}" />
             <parent link="chassis_link" />
-            <child link="range_${name}_link" />
+            <child link="${name}_link" />
         </joint>
-        <link name="range_${name}_link">
+        <link name="${name}_link">
             <collision>
                 <origin xyz="0 0 0" rpy="0 0 0" />
@@ -93,8 +93,9 @@
             </inertial>
         </link>
-        <gazebo reference="range_${name}_link">
+        <gazebo reference="${name}_link">
             <material>Gazebo/Blue</material>
-            <sensor type="ray" name="range_${name}">
-                <update_rate>10</update_rate>
+            <sensor type="ray" name="${name}_sensor">
+                <always_on>true</always_on>
+                <update_rate>30</update_rate>
                 <ray>
                     <range>
@@ -119,5 +120,49 @@
                     <gaussianNoise>0.000</gaussianNoise>
                     <topicName>$(arg ns)/${name}</topicName>
-                    <frameId>range_${name}_link</frameId>
+                    <frameId>${name}_link</frameId>
+                </plugin>
+            </sensor>
+        </gazebo>
+    </macro>
+    <!-- FIXME: Fails unless connected to world frame, I think... -->
+    <macro name="sensor_bump" params="name linX linY linZ angR angP angY">
+        <!-- TODO: Macro these reusable joint templates -->
+        <joint name="${name}_joint" type="fixed">
+            <axis xyz="0 1 0" />
+            <origin xyz="${linX} ${linY} ${linZ}" rpy="${angR} ${angP} ${angY}" />
+            <parent link="chassis_link" />
+            <child link="${name}_link" />
+        </joint>
+        <link name="${name}_link">
+            <collision name="${name}_link_collision">
+                <origin xyz="0 0 0" rpy="0 0 0" />
+                <geometry>
+                    <box size="0.01 0.10 0.01" />
+                </geometry>
+            </collision>
+            <visual>
+                <origin xyz="0 0 0" rpy="0 0 0" />
+                <geometry>
+                    <box size="0.01 0.10 0.01" />
+                </geometry>
+                <material name="blue" />
+            </visual>
+            <inertial>
+                <mass value="0.005" />
+                <origin xyz="0 0 0" rpy="0 0 0" />
+                <box_inertia m="0.005" x="0.01" y="0.10" z="0.01" />
+            </inertial>
+        </link>
+        <gazebo reference="${name}_link">
+            <material>Gazebo/Blue</material>
+            <sensor type="foo" name="${name}_sensor">
+                <always_on>true</always_on>
+                <update_rate>30.0</update_rate>
+                <contact>
+                    <collision>${name}_link_collision</collision>
+                </contact>
+                <plugin name="gazebo_ros_bumper_${name}" filename="libgazebo_ros_bumper.so">
+                    <bumperTopicName>$(arg ns)/${name}</bumperTopicName>
+                    <frameName>${name}_link</frameName>
                 </plugin>
             </sensor>

Commit message: Sensors for DQN

File: kulbu_description/urdf/kulbu.xacro (robot description, xacro)
@@ -182,5 +182,5 @@
     <joint name="laser_joint" type="fixed">
         <axis xyz="0 1 0" />
-        <origin xyz="${chassisLength/2} 0 ${chassisHeight+0.2}" rpy="0 0 0"/><!-- ${PI/2} -->
+        <origin xyz="${chassisLength/4} 0 ${chassisHeight+0.1}" rpy="0 0 0"/><!-- ${PI/2} -->
         <parent link="chassis_link"/>
         <child link="laser_link"/>
@@ -214,11 +214,12 @@
     0.785398163 = 45deg
     -->
-    <sensor_range name="range_0"  linX="${0.02+chassisLength/2}" linY="0"     linZ="${chassisHeight+0.3}" angR="0" angP="0" angY="0" />
-    <sensor_range name="range_1l" linX="${0.02+chassisLength/2}" linY="0.05"  linZ="${chassisHeight+0.3}" angR="0" angP="0" angY="0.261799388" />
-    <sensor_range name="range_2l" linX="${0.02+chassisLength/2}" linY="0.10"  linZ="${chassisHeight+0.3}" angR="0" angP="0" angY="0.523598776" />
-    <sensor_range name="range_3l" linX="${0.02+chassisLength/2}" linY="0.15"  linZ="${chassisHeight+0.3}" angR="0" angP="0" angY="0.785398163" />
-    <sensor_range name="range_1r" linX="${0.02+chassisLength/2}" linY="-0.05" linZ="${chassisHeight+0.3}" angR="0" angP="0" angY="-0.261799388" />
-    <sensor_range name="range_2r" linX="${0.02+chassisLength/2}" linY="-0.10" linZ="${chassisHeight+0.3}" angR="0" angP="0" angY="-0.523598776" />
-    <sensor_range name="range_3r" linX="${0.02+chassisLength/2}" linY="-0.15" linZ="${chassisHeight+0.3}" angR="0" angP="0" angY="-0.785398163" />
+    <!--sensor_range name="range"    linX="${0.02+chassisLength/2}" linY="0"     linZ="${chassisHeight+0.3}" angR="0" angP="0" angY="-3.0" /-->
+    <sensor_range name="range_0"  linX="${chassisLength/2}" linY="0"     linZ="${chassisHeight+0.3}" angR="0" angP="0" angY="0" />
+    <sensor_range name="range_1l" linX="${chassisLength/2}" linY="0.05"  linZ="${chassisHeight+0.3}" angR="0" angP="0" angY="0.261799388" />
+    <sensor_range name="range_2l" linX="${chassisLength/2}" linY="0.10"  linZ="${chassisHeight+0.3}" angR="0" angP="0" angY="0.523598776" />
+    <sensor_range name="range_3l" linX="${chassisLength/2}" linY="0.15"  linZ="${chassisHeight+0.3}" angR="0" angP="0" angY="0.785398163" />
+    <sensor_range name="range_1r" linX="${chassisLength/2}" linY="-0.05" linZ="${chassisHeight+0.3}" angR="0" angP="0" angY="-0.261799388" />
+    <sensor_range name="range_2r" linX="${chassisLength/2}" linY="-0.10" linZ="${chassisHeight+0.3}" angR="0" angP="0" angY="-0.523598776" />
+    <sensor_range name="range_3r" linX="${chassisLength/2}" linY="-0.15" linZ="${chassisHeight+0.3}" angR="0" angP="0" angY="-0.785398163" />
     <!--sensor_bump name="bump_l" linX="${chassisLength/2}" linY="0.15"  linZ="${chassisHeight}" angR="0" angP="0" angY="0.785398163" /-->
     <!--sensor_bump name="bump_r" linX="${chassisLength/2}" linY="-0.15" linZ="${chassisHeight}" angR="0" angP="0" angY="-0.785398163" /-->

File: kulbu_description/urdf/macros.xacro (robot description, xacro)
@@ -97,5 +97,5 @@
             <sensor type="ray" name="${name}_sensor">
                 <always_on>true</always_on>
-                <update_rate>30</update_rate>
+                <update_rate>15.0</update_rate>
                 <ray>
                     <range>
@@ -104,12 +104,13 @@
                         <resolution>0.01</resolution>
                     </range>
+                    <!-- 15deg, 6 samples, reduce glitching. FIXME: What is glitching? Framerate? -->
                     <scan>
                         <horizontal>
-                            <samples>1</samples>
+                            <samples>6</samples>
                             <min_angle>-0.130899694</min_angle>
                             <max_angle>0.130899694</max_angle>
                         </horizontal>
                         <vertical>
-                            <samples>1</samples>
+                            <samples>6</samples>
                             <min_angle>-0.130899694</min_angle>
                             <max_angle>0.130899694</max_angle>
@@ -156,7 +157,7 @@
         <gazebo reference="${name}_link">
             <material>Gazebo/Blue</material>
-            <sensor type="foo" name="${name}_sensor">
+            <sensor type="contact" name="${name}_sensor">
                 <always_on>true</always_on>
-                <update_rate>30.0</update_rate>
+                <update_rate>15.0</update_rate>
                 <contact>
                     <collision>${name}_link_collision</collision>
