Commit message: Updated to gazebo range and added second bot

File: kulbu_description/urdf/kulbu.xacro (robot description, xacro)
@@ -214,12 +214,12 @@
     0.785398163 = 45deg
     -->
-    <!--sensor_range name="range"    linX="${0.02+chassisLength/2}" linY="0"     linZ="${chassisHeight+0.3}" angR="0" angP="0" angY="-3.0" /-->
-    <sensor_range name="range_0"  linX="${chassisLength/2}" linY="0"     linZ="${chassisHeight+0.3}" angR="0" angP="0" angY="0" />
-    <sensor_range name="range_1l" linX="${chassisLength/2}" linY="0.05"  linZ="${chassisHeight+0.3}" angR="0" angP="0" angY="0.261799388" />
-    <sensor_range name="range_2l" linX="${chassisLength/2}" linY="0.10"  linZ="${chassisHeight+0.3}" angR="0" angP="0" angY="0.523598776" />
-    <sensor_range name="range_3l" linX="${chassisLength/2}" linY="0.15"  linZ="${chassisHeight+0.3}" angR="0" angP="0" angY="0.785398163" />
-    <sensor_range name="range_1r" linX="${chassisLength/2}" linY="-0.05" linZ="${chassisHeight+0.3}" angR="0" angP="0" angY="-0.261799388" />
-    <sensor_range name="range_2r" linX="${chassisLength/2}" linY="-0.10" linZ="${chassisHeight+0.3}" angR="0" angP="0" angY="-0.523598776" />
-    <sensor_range name="range_3r" linX="${chassisLength/2}" linY="-0.15" linZ="${chassisHeight+0.3}" angR="0" angP="0" angY="-0.785398163" />
+    <!--sensor_hector_range name="range"    linX="${0.02+chassisLength/2}" linY="0"     linZ="${chassisHeight+0.3}" angR="0" angP="0" angY="-3.0" /-->
+    <sensor_hector_range name="range_0"  linX="${chassisLength/2}" linY="0"     linZ="${chassisHeight+0.3}" angR="0" angP="0" angY="0" />
+    <sensor_hector_range name="range_1l" linX="${chassisLength/2}" linY="0.05"  linZ="${chassisHeight+0.3}" angR="0" angP="0" angY="0.261799388" />
+    <sensor_hector_range name="range_2l" linX="${chassisLength/2}" linY="0.10"  linZ="${chassisHeight+0.3}" angR="0" angP="0" angY="0.523598776" />
+    <sensor_hector_range name="range_3l" linX="${chassisLength/2}" linY="0.15"  linZ="${chassisHeight+0.3}" angR="0" angP="0" angY="0.785398163" />
+    <sensor_hector_range name="range_1r" linX="${chassisLength/2}" linY="-0.05" linZ="${chassisHeight+0.3}" angR="0" angP="0" angY="-0.261799388" />
+    <sensor_hector_range name="range_2r" linX="${chassisLength/2}" linY="-0.10" linZ="${chassisHeight+0.3}" angR="0" angP="0" angY="-0.523598776" />
+    <sensor_hector_range name="range_3r" linX="${chassisLength/2}" linY="-0.15" linZ="${chassisHeight+0.3}" angR="0" angP="0" angY="-0.785398163" />
     <!--sensor_bump name="bump_l" linX="${chassisLength/2}" linY="0.15"  linZ="${chassisHeight}" angR="0" angP="0" angY="0.785398163" /-->
     <!--sensor_bump name="bump_r" linX="${chassisLength/2}" linY="-0.15" linZ="${chassisHeight}" angR="0" angP="0" angY="-0.785398163" /-->

File: kulbu_description/urdf/macros.xacro (robot description, xacro)
@@ -66,5 +66,70 @@
         </transmission>
     </macro>
-    <macro name="sensor_range" params="name linX linY linZ angR angP angY">
+    <macro name="sensor_gazebo_range" params="name linX linY linZ angR angP angY">
+        <joint name="${name}_joint" type="fixed">
+            <axis xyz="0 1 0" />
+            <origin xyz="${linX} ${linY} ${linZ}" rpy="${angR} ${angP} ${angY}" />
+            <parent link="chassis_link" />
+            <child link="${name}_link" />
+        </joint>
+        <link name="${name}_link">
+            <collision>
+                <origin xyz="0 0 0" rpy="0 0 0" />
+                <geometry>
+                    <box size="0.0 0.0 0.0" />
+                </geometry>
+            </collision>
+            <visual>
+                <origin xyz="0 0 0" rpy="0 0 0" />
+                <geometry>
+                    <box size="0.015 0.045 0.02" />
+                </geometry>
+                <material name="blue" />
+            </visual>
+            <inertial>
+                <mass value="0.001" />
+                <origin xyz="0 0 0" rpy="0 0 0" />
+                <inertia ixx="0.000000017" ixy="0" ixz="0" iyy="0.000000017" iyz="0" izz="0.000000017" />
+            </inertial>
+        </link>
+        <gazebo reference="${name}_link">
+            <material>Gazebo/Blue</material>
+            <sensor type="ray" name="${name}_sensor">
+                <always_on>true</always_on>
+                <update_rate>5.0</update_rate>
+                <ray>
+                    <range>
+                        <min>0.02</min>
+                        <max>4.00</max>
+                        <resolution>0.01</resolution>
+                    </range>
+                    <scan>
+                      <horizontal>
+                        <samples>5</samples>
+                        <resolution>1.0</resolution>
+                        <min_angle>-0.130899694</min_angle>
+                        <max_angle>0.130899694</max_angle>
+                      </horizontal>
+                      <vertical>
+                        <samples>5</samples>
+                        <resolution>1</resolution>
+                        <min_angle>-0.130899694</min_angle>
+                        <max_angle>0.130899694</max_angle>
+                      </vertical>
+                    </scan>
+                  </ray>
+                  <plugin filename="libgazebo_ros_range.so" name="gazebo_ros_range">
+                    <gaussianNoise>0.005</gaussianNoise>
+                    <alwaysOn>true</alwaysOn>
+                    <updateRate>5</updateRate>
+                    <topicName>$(arg ns)/${name}</topicName>
+                    <frameName>${name}_link</frameName>
+                    <fov>0.5</fov>
+                    <radiation>ultrasound</radiation>
+                  </plugin>
+            </sensor>
+        </gazebo>
+    </macro>
+    <macro name="sensor_hector_range" params="name linX linY linZ angR angP angY">
         <joint name="${name}_joint" type="fixed">
             <axis xyz="0 1 0" />
