Commit message: Kulbabu definition

File: kulbu_description/urdf/macros.xacro (robot description, xacro)
@@ -83,5 +83,5 @@
                 <origin xyz="0 0 0" rpy="0 0 0" />
                 <geometry>
-                    <box size="0.015 0.045 0.02" />
+                    <box size="0.015 0.015 0.045" />
                 </geometry>
                 <material name="blue" />

Commit message: Unique name for plugin and collision box

File: kulbu_description/urdf/macros.xacro (robot description, xacro)
@@ -77,5 +77,5 @@
                 <origin xyz="0 0 0" rpy="0 0 0" />
                 <geometry>
-                    <box size="0.0 0.0 0.0" />
+                    <box size="0.015 0.015 0.045" />
                 </geometry>
             </collision>
@@ -119,5 +119,6 @@
                     </scan>
                   </ray>
-                  <plugin filename="libgazebo_ros_range.so" name="gazebo_ros_range">
+                  <plugin filename="libgazebo_ros_range.so" name="gazebo_ros_range_${name}">
+                    <robotNamespace>$(arg ns)</robotNamespace>
                     <gaussianNoise>0.005</gaussianNoise>
                     <alwaysOn>true</alwaysOn>
