Commit message: Fix depends and a bunch of stuff

File: kulbu_description/urdf/kulbabu.xacro (robot description, xacro)
@@ -11,4 +11,8 @@
     <xacro:property name="wheelMass" value="5"/>
     <xacro:property name="casterRadius" value="0.015"/>
+    <xacro:property name="bumperHeight" value="0.020"/>
+    <xacro:property name="bumperLength" value="${0.70710678118*chassisLength}"/>
+    <xacro:property name="bumperWidth" value="${0.70710678118*chassisWidth}"/>
+    <xacro:property name="bumperMass" value="5"/>
     <arg name="gui" value="true"/>
     <xacro:include filename="$(find kulbu_description)/urdf/kulbabu.gazebo" />
@@ -77,30 +81,66 @@
         <child link="caster_link"/>
     </joint>
+    <link name='bumper_link'>
+        <collision name='bumper_collision'>
+            <origin xyz="${bumperLength-chassisLength/2} 0 ${wheelRadius+bumperHeight/2}" rpy="0 0 ${45*(PI/180)}" />
+            <geometry>
+                <box size="${bumperLength} ${bumperWidth} ${bumperHeight}"/>
+            </geometry>
+            <surface>
+                <friction>
+                    <ode>
+                        <mu>0</mu>
+                        <mu2>0</mu2>
+                        <slip1>1.0</slip1>
+                        <slip2>1.0</slip2>
+                    </ode>
+                </friction>
+            </surface>
+        </collision>
+        <visual name='bumper_visual'>
+            <origin xyz="${bumperLength-chassisLength/2} 0 ${wheelRadius+bumperHeight/2}" rpy="0 0 ${45*(PI/180)}" />
+            <geometry>
+                <box size="${bumperLength} ${bumperWidth} ${bumperHeight}"/>
+            </geometry>
+            <material name="yellow"/>
+        </visual>
+    </link>
+    <gazebo reference="bumper_link">
+        <mu1 value="0"/>
+        <mu2 value="0"/>
+        <kp  value="10000000.0" />
+        <kd  value="1.0" />
+        <fdir1 value="0 0 0"/>
+        <material>Gazebo/Yellow</material>
+    </gazebo>
+    <joint name="bumper_joint" type="fixed">
+        <parent link="chassis_link"/>
+        <child link="bumper_link"/>
+    </joint>
     <!-- EffortJointInterface/VelocityJointInterface -->
-    <wheel fb="mid"   lr="left"  tX="0"  tY="1"   mu="0.3" interface="VelocityJointInterface" />
-    <wheel fb="mid"   lr="right" tX="0"  tY="-1"  mu="0.3" interface="VelocityJointInterface" />
+    <wheel fb="mid"   lr="left"  tX="0"  tY="0.75"   mu="0.3" interface="VelocityJointInterface" />
+    <wheel fb="mid"   lr="right" tX="0"  tY="-0.75"  mu="0.3" interface="VelocityJointInterface" />
     <!-- Range
     https://jsfiddle.net/MrYellow/2fdtnsbw/
-    -2.356194490 -135 -0.056568542494923796 -0.05656854249492381
-    -1.832595715 -105 -0.02070552360820167 -0.07727406610312547
-    -1.308996939 -75 0.02070552360820166 -0.07727406610312547
-    -0.785398163 -45 0.05656854249492381 -0.056568542494923796
-    -0.261799388 -15 0.07727406610312545 -0.020705523608201673
-    0.261799388 15 0.07727406610312547 0.02070552360820164
-    0.785398163 45 0.056568542494923824 0.05656854249492378
-    1.308996939 75 0.02070552360820171 0.07727406610312545
-    1.832595715 105 -0.02070552360820163 0.07727406610312547
-    2.356194490 135 -0.056568542494923796 0.05656854249492381
-    2.879793266 165 -0.07727406610312547 0.020705523608201645
-    3.403392041 195 -0.07727406610312545 -0.020705523608201694
+    -2.356194490 -135 -0.05126524163602469 -0.051265241636024694
+    -1.832595715 -105 -0.01876438076993276 -0.07002962240595745
+    -1.308996939 -75 0.018764380769932754 -0.07002962240595745
+    -0.785398163 -45 0.051265241636024694 -0.05126524163602469
+    -0.261799388 -15 0.07002962240595743 -0.018764380769932764
+    0.261799388 15 0.07002962240595745 0.018764380769932733
+    0.785398163 45 0.05126524163602471 0.051265241636024673
+    1.308996939 75 0.018764380769932802 0.07002962240595743
+    1.832595715 105 -0.01876438076993273 0.07002962240595746
+    2.356194490 135 -0.05126524163602469 0.051265241636024694
+    2.879793266 165 -0.07002962240595745 0.01876438076993274
     -->
-    <sensor_gazebo_range name="range_1l" linX="0.07727406610312547"  linY="0.02070552360820164" linZ="${0.045+wheelRadius+chassisHeight/2}" angR="0" angP="0" angY="0.261799388" />
-    <sensor_gazebo_range name="range_2l" linX="0.056568542494923824" linY="0.05656854249492378" linZ="${0.045+wheelRadius+chassisHeight/2}" angR="0" angP="0" angY="0.785398163" />
-    <sensor_gazebo_range name="range_3l" linX="0.02070552360820171"  linY="0.07727406610312545" linZ="${0.045+wheelRadius+chassisHeight/2}" angR="0" angP="0" angY="1.308996939" />
-    <sensor_gazebo_range name="range_4l" linX="-0.02070552360820163" linY="0.07727406610312547" linZ="${0.045+wheelRadius+chassisHeight/2}" angR="0" angP="0" angY="1.832595715" />
-    <sensor_gazebo_range name="range_1r" linX="0.07727406610312547"  linY="-0.02070552360820164" linZ="${0.045+wheelRadius+chassisHeight/2}" angR="0" angP="0" angY="-0.261799388" />
-    <sensor_gazebo_range name="range_2r" linX="0.056568542494923824" linY="-0.05656854249492378" linZ="${0.045+wheelRadius+chassisHeight/2}" angR="0" angP="0" angY="-0.785398163" />
-    <sensor_gazebo_range name="range_3r" linX="0.02070552360820171"  linY="-0.07727406610312545" linZ="${0.045+wheelRadius+chassisHeight/2}" angR="0" angP="0" angY="-1.308996939" />
-    <sensor_gazebo_range name="range_4r" linX="-0.02070552360820163" linY="-0.07727406610312547" linZ="${0.045+wheelRadius+chassisHeight/2}" angR="0" angP="0" angY="-1.832595715" />
+    <sensor_gazebo_range name="range_1l" linX="0.07002962240595745"   linY="0.018764380769932733"  linZ="${0.045+wheelRadius+chassisHeight/2}" angR="0" angP="0" angY="0.261799388" />
+    <sensor_gazebo_range name="range_2l" linX="0.05126524163602471"   linY="0.051265241636024673"  linZ="${0.045+wheelRadius+chassisHeight/2}" angR="0" angP="0" angY="0.785398163" />
+    <sensor_gazebo_range name="range_3l" linX="0.018764380769932802"  linY="0.07002962240595745"   linZ="${0.045+wheelRadius+chassisHeight/2}" angR="0" angP="0" angY="1.308996939" />
+    <sensor_gazebo_range name="range_4l" linX="-0.01876438076993273"  linY="0.07002962240595745"   linZ="${0.045+wheelRadius+chassisHeight/2}" angR="0" angP="0" angY="1.832595715" />
+    <sensor_gazebo_range name="range_1r" linX="0.07002962240595745"   linY="-0.018764380769932733" linZ="${0.045+wheelRadius+chassisHeight/2}" angR="0" angP="0" angY="-0.261799388" />
+    <sensor_gazebo_range name="range_2r" linX="0.05126524163602471"   linY="-0.051265241636024673" linZ="${0.045+wheelRadius+chassisHeight/2}" angR="0" angP="0" angY="-0.785398163" />
+    <sensor_gazebo_range name="range_3r" linX="0.018764380769932802"  linY="-0.07002962240595745"  linZ="${0.045+wheelRadius+chassisHeight/2}" angR="0" angP="0" angY="-1.308996939" />
+    <sensor_gazebo_range name="range_4r" linX="-0.01876438076993273"  linY="-0.07002962240595745"  linZ="${0.045+wheelRadius+chassisHeight/2}" angR="0" angP="0" angY="-1.832595715" />
     <!--sensor_bump name="bump_l" linX="${chassisLength/2}" linY="0.15"  linZ="${chassisHeight}" angR="0" angP="0" angY="0.785398163" /-->
     <!--sensor_bump name="bump_r" linX="${chassisLength/2}" linY="-0.15" linZ="${chassisHeight}" angR="0" angP="0" angY="-0.785398163" /-->

File: kulbu_description/urdf/macros.xacro (robot description, xacro)
@@ -100,5 +100,5 @@
                 <ray>
                     <range>
-                        <min>0.02</min>
+                        <min>0.01</min>
                         <max>4.00</max>
                         <resolution>0.01</resolution>

Commit message: Gazebo 2.x has issues with multiple bumpers

File: kulbu_description/urdf/kulbabu.xacro (robot description, xacro)
@@ -81,5 +81,5 @@
         <child link="caster_link"/>
     </joint>
-    <link name='bumper_link'>
+    <!--link name='bumper_link'>
         <collision name='bumper_collision'>
             <origin xyz="${bumperLength-chassisLength/2} 0 ${wheelRadius+bumperHeight/2}" rpy="0 0 ${45*(PI/180)}" />
@@ -117,5 +117,5 @@
         <parent link="chassis_link"/>
         <child link="bumper_link"/>
-    </joint>
+    </joint-->
     <!-- EffortJointInterface/VelocityJointInterface -->
     <wheel fb="mid"   lr="left"  tX="0"  tY="0.75"   mu="0.3" interface="VelocityJointInterface" />
@@ -143,6 +143,6 @@
     <sensor_gazebo_range name="range_3r" linX="0.018764380769932802"  linY="-0.07002962240595745"  linZ="${0.045+wheelRadius+chassisHeight/2}" angR="0" angP="0" angY="-1.308996939" />
     <sensor_gazebo_range name="range_4r" linX="-0.01876438076993273"  linY="-0.07002962240595745"  linZ="${0.045+wheelRadius+chassisHeight/2}" angR="0" angP="0" angY="-1.832595715" />
-    <!--sensor_bump name="bump_l" linX="${chassisLength/2}" linY="0.15"  linZ="${chassisHeight}" angR="0" angP="0" angY="0.785398163" /-->
-    <!--sensor_bump name="bump_r" linX="${chassisLength/2}" linY="-0.15" linZ="${chassisHeight}" angR="0" angP="0" angY="-0.785398163" /-->
+    <!--sensor_bump name="bump_l" linX="${0.045+chassisLength/4}" linY="${chassisLength/4}"  linZ="${chassisHeight/2}" angR="0" angP="0" angY="${45*(PI/180)}" />
+    <sensor_bump name="bump_r" linX="${0.045+chassisLength/4}" linY="-${chassisLength/4}" linZ="${chassisHeight/2}" angR="0" angP="0" angY="-${45*(PI/180)}" /-->
     <!-- IMU -->
     <joint name="imu_joint" type="fixed">

File: kulbu_description/urdf/macros.xacro (robot description, xacro)
@@ -212,5 +212,5 @@
                     <box size="0.01 0.10 0.01" />
                 </geometry>
-                <material name="blue" />
+                <material name="yellow" />
             </visual>
             <inertial>
@@ -220,6 +220,6 @@
             </inertial>
         </link>
-        <gazebo reference="${name}_link">
-            <material>Gazebo/Blue</material>
+        <!--gazebo reference="${name}_link">
+            <material>Gazebo/Yellow</material>
             <sensor type="contact" name="${name}_sensor">
                 <always_on>true</always_on>
@@ -233,5 +233,5 @@
                 </plugin>
             </sensor>
-        </gazebo>
+        </gazebo-->
     </macro>
 </robot>

Commit message: Fix box size

File: kulbu_description/urdf/kulbabu.xacro (robot description, xacro)
@@ -136,5 +136,5 @@
     -->
     <sensor_gazebo_range name="range_1l" linX="0.07002962240595745"   linY="0.018764380769932733"  linZ="${0.045+wheelRadius+chassisHeight/2}" angR="0" angP="0" angY="0.261799388" />
-    <sensor_gazebo_range name="range_2l" linX="0.05126524163602471"   linY="0.051265241636024673"  linZ="${0.045+wheelRadius+chassisHeight/2}" angR="0" angP="0" angY="0.785398163" />
+    <!--sensor_gazebo_range name="range_2l" linX="0.05126524163602471"   linY="0.051265241636024673"  linZ="${0.045+wheelRadius+chassisHeight/2}" angR="0" angP="0" angY="0.785398163" />
     <sensor_gazebo_range name="range_3l" linX="0.018764380769932802"  linY="0.07002962240595745"   linZ="${0.045+wheelRadius+chassisHeight/2}" angR="0" angP="0" angY="1.308996939" />
     <sensor_gazebo_range name="range_4l" linX="-0.01876438076993273"  linY="0.07002962240595745"   linZ="${0.045+wheelRadius+chassisHeight/2}" angR="0" angP="0" angY="1.832595715" />
@@ -142,5 +142,5 @@
     <sensor_gazebo_range name="range_2r" linX="0.05126524163602471"   linY="-0.051265241636024673" linZ="${0.045+wheelRadius+chassisHeight/2}" angR="0" angP="0" angY="-0.785398163" />
     <sensor_gazebo_range name="range_3r" linX="0.018764380769932802"  linY="-0.07002962240595745"  linZ="${0.045+wheelRadius+chassisHeight/2}" angR="0" angP="0" angY="-1.308996939" />
-    <sensor_gazebo_range name="range_4r" linX="-0.01876438076993273"  linY="-0.07002962240595745"  linZ="${0.045+wheelRadius+chassisHeight/2}" angR="0" angP="0" angY="-1.832595715" />
+    <sensor_gazebo_range name="range_4r" linX="-0.01876438076993273"  linY="-0.07002962240595745"  linZ="${0.045+wheelRadius+chassisHeight/2}" angR="0" angP="0" angY="-1.832595715" /-->
     <!--sensor_bump name="bump_l" linX="${0.045+chassisLength/4}" linY="${chassisLength/4}"  linZ="${chassisHeight/2}" angR="0" angP="0" angY="${45*(PI/180)}" />
     <sensor_bump name="bump_r" linX="${0.045+chassisLength/4}" linY="-${chassisLength/4}" linZ="${chassisHeight/2}" angR="0" angP="0" angY="-${45*(PI/180)}" /-->
@@ -156,5 +156,5 @@
             <origin xyz="0 0 ${chassisHeight}" rpy="0 0 0"/>
             <geometry>
-                <box size="0.0 0.0 0.0"/>
+                <box size="0.01 0.01 0.01"/>
             </geometry>
         </collision>

File: kulbu_description/urdf/macros.xacro (robot description, xacro)
@@ -95,5 +95,5 @@
         <gazebo reference="${name}_link">
             <material>Gazebo/Blue</material>
-            <sensor type="ray" name="${name}_sensor">
+            <!--sensor type="ray" name="${name}_sensor">
                 <always_on>true</always_on>
                 <update_rate>5.0</update_rate>
@@ -129,5 +129,5 @@
                     <radiation>ultrasound</radiation>
                   </plugin>
-            </sensor>
+            </sensor-->
         </gazebo>
     </xacro:macro>

Commit message: Enable some sensors disable others

File: kulbu_description/urdf/kulbabu.xacro (robot description, xacro)
@@ -143,8 +143,8 @@
     <sensor_gazebo_range name="range_3r" linX="0.018764380769932802"  linY="-0.07002962240595745"  linZ="${0.045+wheelRadius+chassisHeight/2}" angR="0" angP="0" angY="-1.308996939" />
     <sensor_gazebo_range name="range_4r" linX="-0.01876438076993273"  linY="-0.07002962240595745"  linZ="${0.045+wheelRadius+chassisHeight/2}" angR="0" angP="0" angY="-1.832595715" />
-    <!--sensor_bump name="bump_l" linX="${0.045+chassisLength/4}" linY="${chassisLength/4}"  linZ="${chassisHeight/2}" angR="0" angP="0" angY="${45*(PI/180)}" />
-    <sensor_bump name="bump_r" linX="${0.045+chassisLength/4}" linY="-${chassisLength/4}" linZ="${chassisHeight/2}" angR="0" angP="0" angY="-${45*(PI/180)}" /-->
+    <sensor_bump name="bump_l" linX="${0.045+chassisLength/4}" linY="${chassisLength/4}"  linZ="${chassisHeight/2}" angR="0" angP="0" angY="${45*(PI/180)}" />
+    <sensor_bump name="bump_r" linX="${0.045+chassisLength/4}" linY="-${chassisLength/4}" linZ="${chassisHeight/2}" angR="0" angP="0" angY="-${45*(PI/180)}" />
     <!-- IMU -->
-    <joint name="imu_joint" type="fixed">
+    <!--joint name="imu_joint" type="fixed">
         <axis xyz="0 1 0" />
         <origin xyz="0 0 0" rpy="0 0 0"/>
@@ -171,4 +171,4 @@
             <inertia ixx="1e-6" ixy="0" ixz="0" iyy="1e-6" iyz="0" izz="1e-6" />
         </inertial>
-    </link>
+    </link-->
 </robot>

File: kulbu_description/urdf/macros.xacro (robot description, xacro)
@@ -119,5 +119,5 @@
                     </scan>
                   </ray>
-                  <plugin filename="libgazebo_ros_range.so" name="gazebo_ros_range_${name}">
+                  <plugin name="gazebo_ros_range_${name}" filename="libgazebo_ros_range.so">
                     <robotNamespace>$(arg ns)</robotNamespace>
                     <gaussianNoise>0.005</gaussianNoise>
@@ -185,4 +185,5 @@
                 </ray>
                 <plugin name="gazebo_ros_sonar_${name}_controller" filename="libhector_gazebo_ros_sonar.so">
+                    <robotNamespace>$(arg ns)</robotNamespace>
                     <gaussianNoise>0.000</gaussianNoise>
                     <topicName>$(arg ns)/${name}</topicName>
@@ -221,5 +222,5 @@
             </inertial>
         </link>
-        <!--gazebo reference="${name}_link">
+        <gazebo reference="${name}_link">
             <material>Gazebo/Yellow</material>
             <sensor type="contact" name="${name}_sensor">
@@ -230,9 +231,10 @@
                 </contact>
                 <plugin name="gazebo_ros_bumper_${name}" filename="libgazebo_ros_bumper.so">
+                    <robotNamespace>$(arg ns)</robotNamespace>
                     <bumperTopicName>$(arg ns)/${name}</bumperTopicName>
                     <frameName>${name}_link</frameName>
                 </plugin>
             </sensor>
-        </gazebo-->
+        </gazebo>
     </xacro:macro>
 </robot>

Commit message: Tidy up model and fix masses

File: kulbu_description/urdf/kulbabu.xacro (robot description, xacro)
@@ -5,14 +5,15 @@
     <xacro:property name="chassisLength" value="0.160"/>
     <xacro:property name="chassisWidth" value="0.160"/>
-    <xacro:property name="chassisMass" value="50"/>
+    <xacro:property name="chassisMass" value="10"/>
     <xacro:property name="wheelWidth" value="0.025"/>
     <xacro:property name="wheelRadius" value="0.030"/>
     <xacro:property name="wheelPos" value="0.2"/>
-    <xacro:property name="wheelMass" value="5"/>
+    <xacro:property name="wheelMass" value="2"/>
     <xacro:property name="casterRadius" value="0.015"/>
+    <xacro:property name="casterMass" value="1"/>
     <xacro:property name="bumperHeight" value="0.020"/>
     <xacro:property name="bumperLength" value="${0.70710678118*chassisLength}"/>
     <xacro:property name="bumperWidth" value="${0.70710678118*chassisWidth}"/>
-    <xacro:property name="bumperMass" value="5"/>
+    <xacro:property name="bumperMass" value="0.5"/>
     <xacro:arg name="gui" default="true"/>
     <xacro:include filename="$(find kulbu_description)/urdf/kulbabu.gazebo" />
@@ -39,5 +40,5 @@
         </visual>
         <inertial>
-            <origin xyz="${-chassisLength/8} 0 ${-0.015+wheelRadius+chassisHeight/2}" rpy="0 0 0"/>
+            <origin xyz="0 0 ${-0.015+wheelRadius+chassisHeight/2}" rpy="0 0 0"/>
             <mass value="${chassisMass}"/>
             <cylinder_inertia m="${chassisMass}" r="${chassisLength/2}" h="${chassisHeight}"/>
@@ -68,18 +69,15 @@
             <material name="green"/>
         </visual>
+        <inertial>
+            <origin xyz="${casterRadius-chassisLength/2} 0 ${wheelRadius-casterRadius}" rpy="0 0 0" />
+            <mass value="${casterMass}"/>
+            <sphere_inertia m="${casterMass}" r="${casterRadius}"/>
+        </inertial>
     </link>
-    <gazebo reference="caster_link">
-        <mu1 value="0"/>
-        <mu2 value="0"/>
-        <kp  value="10000000.0" />
-        <kd  value="1.0" />
-        <fdir1 value="0 0 0"/>
-        <material>Gazebo/Green</material>
-    </gazebo>
     <joint name="caster_joint" type="fixed">
         <parent link="chassis_link"/>
         <child link="caster_link"/>
     </joint>
-    <!--link name='bumper_link'>
+    <link name='bumper_link'>
         <collision name='bumper_collision'>
             <origin xyz="${bumperLength-chassisLength/2} 0 ${wheelRadius+bumperHeight/2}" rpy="0 0 ${45*(PI/180)}" />
@@ -105,17 +103,14 @@
             <material name="yellow"/>
         </visual>
+        <inertial>
+            <origin xyz="${bumperLength-chassisLength/2} 0 ${wheelRadius+bumperHeight/2}" rpy="0 0 ${45*(PI/180)}" />
+            <mass value="${bumperMass}"/>
+            <box_inertia m="${bumperMass}" x="${bumperLength/2}" y="${bumperLength/2}" z="${bumperHeight/2}"/>
+        </inertial>
     </link>
-    <gazebo reference="bumper_link">
-        <mu1 value="0"/>
-        <mu2 value="0"/>
-        <kp  value="10000000.0" />
-        <kd  value="1.0" />
-        <fdir1 value="0 0 0"/>
-        <material>Gazebo/Yellow</material>
-    </gazebo>
     <joint name="bumper_joint" type="fixed">
         <parent link="chassis_link"/>
         <child link="bumper_link"/>
-    </joint-->
+    </joint>
     <!-- EffortJointInterface/VelocityJointInterface -->
     <wheel fb="mid"   lr="left"  tX="0"  tY="0.75"   mu="0.3" interface="VelocityJointInterface" />
@@ -143,6 +138,6 @@
     <sensor_gazebo_range name="range_3r" linX="0.018764380769932802"  linY="-0.07002962240595745"  linZ="${0.045+wheelRadius+chassisHeight/2}" angR="0" angP="0" angY="-1.308996939" />
     <sensor_gazebo_range name="range_4r" linX="-0.01876438076993273"  linY="-0.07002962240595745"  linZ="${0.045+wheelRadius+chassisHeight/2}" angR="0" angP="0" angY="-1.832595715" />
-    <sensor_bump name="bump_l" linX="${0.045+chassisLength/4}" linY="${chassisLength/4}"  linZ="${chassisHeight/2}" angR="0" angP="0" angY="${45*(PI/180)}" />
-    <sensor_bump name="bump_r" linX="${0.045+chassisLength/4}" linY="-${chassisLength/4}" linZ="${chassisHeight/2}" angR="0" angP="0" angY="-${45*(PI/180)}" />
+    <!--sensor_bump name="bump_l" linX="${0.045+chassisLength/4}" linY="${chassisLength/4}"  linZ="${chassisHeight/2}" angR="0" angP="0" angY="${45*(PI/180)}" />
+    <sensor_bump name="bump_r" linX="${0.045+chassisLength/4}" linY="-${chassisLength/4}" linZ="${chassisHeight/2}" angR="0" angP="0" angY="-${45*(PI/180)}" /-->
     <!-- IMU -->
     <!--joint name="imu_joint" type="fixed">

File: kulbu_description/urdf/macros.xacro (robot description, xacro)
@@ -26,4 +26,14 @@
                   <cylinder length="${wheelWidth}" radius="${wheelRadius}"/>
               </geometry>
+              <surface>
+                <friction>
+                    <ode>
+                        <mu>1000000</mu>
+                        <mu2>100</mu2>
+                        <slip1>0</slip1>
+                        <slip2>0</slip2>
+                    </ode>
+                </friction>
+              </surface>
           </collision>
           <visual>
@@ -41,9 +51,9 @@
         </link>
         <gazebo reference="${fb}_${lr}_wheel">
-            <mu1 value="${mu}"/>
+            <!--mu1 value="${mu}"/>
             <mu2 value="${mu}"/>
             <kp  value="10000000.0" />
             <kd  value="1.0" />
-            <fdir1 value="0 0 0"/>
+            <fdir1 value="0 0 0"/-->
             <material>Gazebo/Black</material>
         </gazebo>
@@ -229,5 +239,5 @@
                 <contact>
                     <collision>${name}_link_collision</collision>
-                    <!--topic>${name}_link_collision</topic-->
+                    <!--topic>${name}_link</topic-->
                 </contact>
                 <plugin name="gazebo_ros_bumper_${name}" filename="libgazebo_ros_bumper.so">
