Commit message: Attempts at fixing friction

File: kulbu_description/urdf/kulbabu.xacro (robot description, xacro)
@@ -52,4 +52,10 @@
             </geometry>
             <surface>
+                <!--contact>
+                    <ode>
+                        <kp>1e+08</kp>
+                        <kd>10000</kd>
+                    </ode>
+                </contact-->
                 <friction>
                     <ode>
@@ -81,9 +87,15 @@
     <link name='bumper_link'>
         <collision name='bumper_collision'>
-            <origin xyz="${bumperLength-chassisLength/2} 0 ${wheelRadius+bumperHeight/2}" rpy="0 0 ${45*(PI/180)}" />
+            <origin xyz="${0.015+bumperLength-chassisLength/2} 0 ${wheelRadius+bumperHeight/2}" rpy="0 0 ${45*(PI/180)}" />
             <geometry>
                 <box size="${bumperLength} ${bumperWidth} ${bumperHeight}"/>
             </geometry>
             <surface>
+                <!--contact>
+                    <ode>
+                        <kp>1e+08</kp>
+                        <kd>10000</kd>
+                    </ode>
+                </contact-->
                 <friction>
                     <ode>
@@ -97,5 +109,5 @@
         </collision>
         <visual name='bumper_visual'>
-            <origin xyz="${bumperLength-chassisLength/2} 0 ${wheelRadius+bumperHeight/2}" rpy="0 0 ${45*(PI/180)}" />
+            <origin xyz="${0.015+bumperLength-chassisLength/2} 0 ${wheelRadius+bumperHeight/2}" rpy="0 0 ${45*(PI/180)}" />
             <geometry>
                 <box size="${bumperLength} ${bumperWidth} ${bumperHeight}"/>
@@ -104,5 +116,5 @@
         </visual>
         <inertial>
-            <origin xyz="${bumperLength-chassisLength/2} 0 ${wheelRadius+bumperHeight/2}" rpy="0 0 ${45*(PI/180)}" />
+            <origin xyz="${0.015+bumperLength-chassisLength/2} 0 ${wheelRadius+bumperHeight/2}" rpy="0 0 ${45*(PI/180)}" />
             <mass value="${bumperMass}"/>
             <box_inertia m="${bumperMass}" x="${bumperLength/2}" y="${bumperLength/2}" z="${bumperHeight/2}"/>

File: kulbu_description/urdf/macros.xacro (robot description, xacro)
@@ -21,41 +21,44 @@
     <xacro:macro name="wheel" params="fb lr tX tY mu interface">
         <link name="${fb}_${lr}_wheel">
-          <collision>
-              <origin xyz="0 0 0" rpy="0 ${PI/2} ${PI/2}" />
-              <geometry>
-                  <cylinder length="${wheelWidth}" radius="${wheelRadius}"/>
-              </geometry>
-              <surface>
-                <friction>
-                    <ode>
-                        <mu>1000000</mu>
-                        <mu2>100</mu2>
-                        <slip1>0</slip1>
-                        <slip2>0</slip2>
-                    </ode>
-                </friction>
-              </surface>
-          </collision>
-          <visual>
-              <origin xyz="0 0 0" rpy="0 ${PI/2} ${PI/2}" />
-              <geometry>
-                  <cylinder length="${wheelWidth}" radius="${wheelRadius}"/>
-              </geometry>
-              <material name="black"/>
-          </visual>
-          <inertial>
-              <origin xyz="0 0 0" rpy="0 ${PI/2} ${PI/2}" />
-              <mass value="${wheelMass}"/>
-              <cylinder_inertia m="${wheelMass}" r="${wheelRadius}" h="${wheelWidth}"/>
-          </inertial>
+            <collision>
+                <origin xyz="0 0 0" rpy="0 ${PI/2} ${PI/2}" />
+                <geometry>
+                    <cylinder length="${wheelWidth}" radius="${wheelRadius}"/>
+                </geometry>
+                <surface>
+                    <!--contact>
+                        <ode>
+                            <kp>1e+08</kp>
+                            <kd>10000</kd>
+                        </ode>
+                    </contact-->
+                    <friction>
+                        <ode>
+                            <mu>1000000</mu>
+                            <mu2>100</mu2>
+                            <slip1>0</slip1>
+                            <slip2>0</slip2>
+                        </ode>
+                    </friction>
+                </surface>
+            </collision>
+            <visual>
+                <origin xyz="0 0 0" rpy="0 ${PI/2} ${PI/2}" />
+                <geometry>
+                    <cylinder length="${wheelWidth}" radius="${wheelRadius}"/>
+                </geometry>
+                <material name="black"/>
+            </visual>
+            <inertial>
+                <origin xyz="0 0 0" rpy="0 ${PI/2} ${PI/2}" />
+                <mass value="${wheelMass}"/>
+                <cylinder_inertia m="${wheelMass}" r="${wheelRadius}" h="${wheelWidth}"/>
+            </inertial>
         </link>
         <gazebo reference="${fb}_${lr}_wheel">
-            <!--mu1 value="${mu}"/>
-            <mu2 value="${mu}"/>
-            <kp  value="10000000.0" />
-            <kd  value="1.0" />
-            <fdir1 value="0 0 0"/-->
+            <!--mu1>1000000.0</mu1>
+            <mu2>100.0</mu2>
             <kp>1000000.0</kp>
-            <kd>1.0</kd>
+            <kd>1.0</kd-->
             <material>Gazebo/Black</material>
         </gazebo>

Commit message: Place joints before links

File: kulbu_description/urdf/kulbabu.xacro (robot description, xacro)
@@ -45,4 +45,8 @@
         </inertial>
     </link>
+    <joint name="caster_joint" type="fixed">
+        <parent link="chassis_link"/>
+        <child link="caster_link"/>
+    </joint>
     <link name='caster_link'>
         <collision name='caster_collision'>
@@ -81,7 +85,7 @@
         </inertial>
     </link>
-    <joint name="caster_joint" type="fixed">
+    <joint name="bumper_joint" type="fixed">
         <parent link="chassis_link"/>
-        <child link="caster_link"/>
+        <child link="bumper_link"/>
     </joint>
     <link name='bumper_link'>
@@ -121,8 +125,4 @@
         </inertial>
     </link>
-    <joint name="bumper_joint" type="fixed">
-        <parent link="chassis_link"/>
-        <child link="bumper_link"/>
-    </joint>
     <!-- EffortJointInterface/VelocityJointInterface -->
     <wheel fb="mid"   lr="left"  tX="0"  tY="0.75"   mu="0.3" interface="VelocityJointInterface" />

Commit message: Use double quotes consistently

File: kulbu_description/urdf/kulbabu.xacro (robot description, xacro)
@@ -25,5 +25,5 @@
         <child link="chassis_link"/>
     </joint>
-    <link name='chassis_link'>
+    <link name="chassis_link">
         <collision>
             <origin xyz="0 0 ${-0.015+wheelRadius+chassisHeight/2}" rpy="0 0 0"/>
@@ -49,6 +49,6 @@
         <child link="caster_link"/>
     </joint>
-    <link name='caster_link'>
-        <collision name='caster_collision'>
+    <link name="caster_link">
+        <collision name="caster_collision">
             <origin xyz="${casterRadius-chassisLength/2} 0 ${wheelRadius-casterRadius}" rpy="0 0 0" />
             <geometry>
@@ -72,5 +72,5 @@
             </surface>
         </collision>
-        <visual name='caster_visual'>
+        <visual name="caster_visual">
             <origin xyz="${casterRadius-chassisLength/2} 0 ${wheelRadius-casterRadius}" rpy="0 0 0" />
             <geometry>
@@ -89,6 +89,6 @@
         <child link="bumper_link"/>
     </joint>
-    <link name='bumper_link'>
-        <collision name='bumper_collision'>
+    <link name="bumper_link">
+        <collision name="bumper_collision">
             <origin xyz="${0.015+bumperLength-chassisLength/2} 0 ${wheelRadius+bumperHeight/2}" rpy="0 0 ${45*(PI/180)}" />
             <geometry>
@@ -112,5 +112,5 @@
             </surface>
         </collision>
-        <visual name='bumper_visual'>
+        <visual name="bumper_visual">
             <origin xyz="${0.015+bumperLength-chassisLength/2} 0 ${wheelRadius+bumperHeight/2}" rpy="0 0 ${45*(PI/180)}" />
             <geometry>

Commit message: Fx naming issue blocking gazebo refs

File: kulbu_description/urdf/kulbabu.xacro (robot description, xacro)
@@ -50,5 +50,5 @@
     </joint>
     <link name="caster_link">
-        <collision name="caster_collision">
+        <collision>
             <origin xyz="${casterRadius-chassisLength/2} 0 ${wheelRadius-casterRadius}" rpy="0 0 0" />
             <geometry>
@@ -56,10 +56,10 @@
             </geometry>
             <surface>
-                <!--contact>
+                <contact>
                     <ode>
                         <kp>1e+08</kp>
                         <kd>10000</kd>
                     </ode>
-                </contact-->
+                </contact>
                 <friction>
                     <ode>
@@ -72,5 +72,5 @@
             </surface>
         </collision>
-        <visual name="caster_visual">
+        <visual>
             <origin xyz="${casterRadius-chassisLength/2} 0 ${wheelRadius-casterRadius}" rpy="0 0 0" />
             <geometry>
@@ -90,5 +90,5 @@
     </joint>
     <link name="bumper_link">
-        <collision name="bumper_collision">
+        <collision>
             <origin xyz="${0.015+bumperLength-chassisLength/2} 0 ${wheelRadius+bumperHeight/2}" rpy="0 0 ${45*(PI/180)}" />
             <geometry>
@@ -96,10 +96,10 @@
             </geometry>
             <surface>
-                <!--contact>
+                <contact>
                     <ode>
                         <kp>1e+08</kp>
                         <kd>10000</kd>
                     </ode>
-                </contact-->
+                </contact>
                 <friction>
                     <ode>
@@ -112,5 +112,5 @@
             </surface>
         </collision>
-        <visual name="bumper_visual">
+        <visual>
             <origin xyz="${0.015+bumperLength-chassisLength/2} 0 ${wheelRadius+bumperHeight/2}" rpy="0 0 ${45*(PI/180)}" />
             <geometry>

File: kulbu_description/urdf/macros.xacro (robot description, xacro)
@@ -27,10 +27,10 @@
                 </geometry>
                 <surface>
-                    <!--contact>
+                    <contact>
                         <ode>
                             <kp>1e+08</kp>
                             <kd>10000</kd>
                         </ode>
-                    </contact-->
+                    </contact>
                     <friction>
                         <ode>
