Commit message: Update xacro tags

File: kulbu_description/urdf/goal.xacro (robot description, xacro)
@@ -6,5 +6,5 @@
     <xacro:property name="chassisWidth" value="0.25"/>
     <xacro:property name="chassisMass" value="25"/>
-    <arg name="gui" value="true"/>
+    <xacro:arg name="gui" default="true"/>
     <xacro:include filename="$(find kulbu_description)/urdf/materials.xacro" />
     <xacro:include filename="$(find kulbu_description)/urdf/macros.xacro" />

File: kulbu_description/urdf/kulbabu.xacro (robot description, xacro)
@@ -15,5 +15,5 @@
     <xacro:property name="bumperWidth" value="${0.70710678118*chassisWidth}"/>
     <xacro:property name="bumperMass" value="5"/>
-    <arg name="gui" value="true"/>
+    <xacro:arg name="gui" default="true"/>
     <xacro:include filename="$(find kulbu_description)/urdf/kulbabu.gazebo" />
     <xacro:include filename="$(find kulbu_description)/urdf/materials.xacro" />

File: kulbu_description/urdf/kulbu.xacro (robot description, xacro)
@@ -12,5 +12,5 @@
     <xacro:property name="cameraSize" value="0.05"/>
     <xacro:property name="cameraMass" value="0.1"/>
-    <arg name="gui" value="true"/>
+    <xacro:arg name="gui" value="true"/>
     <xacro:include filename="$(find kulbu_description)/urdf/kulbu.gazebo" />
     <xacro:include filename="$(find kulbu_description)/urdf/materials.xacro" />

File: kulbu_description/urdf/macros.xacro (robot description, xacro)
@@ -1,23 +1,23 @@
 <?xml version="1.0"?>
 <robot name="kulbu" xmlns:xacro="http://www.ros.org/wiki/xacro">
-    <macro name="cylinder_inertia" params="m r h">
+    <xacro:macro name="cylinder_inertia" params="m r h">
         <inertia  ixx="${m*(3*r*r+h*h)/12}" ixy="0" ixz="0"
           iyy="${m*(3*r*r+h*h)/12}" iyz="0"
           izz="${m*r*r/2}"
         />
-    </macro>
-    <macro name="box_inertia" params="m x y z">
+    </xacro:macro>
+    <xacro:macro name="box_inertia" params="m x y z">
         <inertia  ixx="${m*(y*y+z*z)/12}" ixy="0" ixz="0"
           iyy="${m*(x*x+z*z)/12}" iyz="0"
           izz="${m*(x*x+z*z)/12}"
         />
-    </macro>
-    <macro name="sphere_inertia" params="m r">
+    </xacro:macro>
+    <xacro:macro name="sphere_inertia" params="m r">
         <inertia  ixx="${2*m*r*r/5}" ixy="0" ixz="0"
           iyy="${2*m*r*r/5}" iyz="0"
           izz="${2*m*r*r/5}"
         />
-    </macro>
-    <macro name="wheel" params="fb lr tX tY mu interface">
+    </xacro:macro>
+    <xacro:macro name="wheel" params="fb lr tX tY mu interface">
         <link name="${fb}_${lr}_wheel">
           <collision>
@@ -65,6 +65,6 @@
             </joint>
         </transmission>
-    </macro>
-    <macro name="sensor_gazebo_range" params="name linX linY linZ angR angP angY">
+    </xacro:macro>
+    <xacro:macro name="sensor_gazebo_range" params="name linX linY linZ angR angP angY">
         <joint name="${name}_joint" type="fixed">
             <axis xyz="0 1 0" />
@@ -130,6 +130,6 @@
             </sensor>
         </gazebo>
-    </macro>
-    <macro name="sensor_hector_range" params="name linX linY linZ angR angP angY">
+    </xacro:macro>
+    <xacro:macro name="sensor_hector_range" params="name linX linY linZ angR angP angY">
         <joint name="${name}_joint" type="fixed">
             <axis xyz="0 1 0" />
@@ -190,7 +190,7 @@
             </sensor>
         </gazebo>
-    </macro>
+    </xacro:macro>
     <!-- FIXME: Fails unless connected to world frame, I think... -->
-    <macro name="sensor_bump" params="name linX linY linZ angR angP angY">
+    <xacro:macro name="sensor_bump" params="name linX linY linZ angR angP angY">
         <!-- TODO: Macro these reusable joint templates -->
         <joint name="${name}_joint" type="fixed">
@@ -234,4 +234,4 @@
             </sensor>
         </gazebo-->
-    </macro>
+    </xacro:macro>
 </robot>

Commit message: No bumper, smaller goal

File: kulbu_description/urdf/goal.xacro (robot description, xacro)
@@ -2,7 +2,7 @@
 <robot name="goal" xmlns:xacro="http://www.ros.org/wiki/xacro">
     <xacro:property name="PI" value="3.1415926535897931"/>
-    <xacro:property name="chassisHeight" value="0.25"/>
-    <xacro:property name="chassisLength" value="0.25"/>
-    <xacro:property name="chassisWidth" value="0.25"/>
+    <xacro:property name="chassisHeight" value="0.1"/>
+    <xacro:property name="chassisLength" value="0.1"/>
+    <xacro:property name="chassisWidth" value="0.1"/>
     <xacro:property name="chassisMass" value="25"/>
     <xacro:arg name="gui" default="true"/>

File: kulbu_description/urdf/kulbabu.xacro (robot description, xacro)
@@ -69,5 +69,5 @@
         </inertial>
     </link>
-    <joint name="bumper_joint" type="fixed">
+    <!--joint name="bumper_joint" type="fixed">
         <parent link="chassis_link"/>
         <child link="bumper_link"/>
@@ -92,5 +92,5 @@
             <box_inertia m="${bumperMass}" x="${bumperLength/2}" y="${bumperLength/2}" z="${bumperHeight/2}"/>
         </inertial>
-    </link>
+    </link-->
     <!-- EffortJointInterface/VelocityJointInterface -->
     <wheel fb="mid"   lr="left"  tX="0"  tY="0.75"   mu="0.3" interface="VelocityJointInterface" />

Commit message: Goal as sphere

File: kulbu_description/urdf/goal.xacro (robot description, xacro)
@@ -18,5 +18,5 @@
             <origin xyz="0 0 0" rpy="0 0 0"/>
             <geometry>
-                <box size="${chassisLength} ${chassisWidth} ${chassisHeight}"/>
+                <sphere radius="${chassisLength}"/>
             </geometry>
         </collision>
@@ -24,5 +24,5 @@
             <origin xyz="0 0 0" rpy="0 0 0"/>
             <geometry>
-                <box size="${chassisLength} ${chassisWidth} ${chassisHeight}"/>
+                <sphere radius="${chassisLength}"/>
             </geometry>
             <material name="green"/>
@@ -31,5 +31,5 @@
             <origin xyz="0 0 0" rpy="0 0 0"/>
             <mass value="${chassisMass}"/>
-            <box_inertia m="${chassisMass}" x="${chassisLength}" y="${chassisWidth}" z="${chassisHeight}"/>
+            <sphere_inertia m="${chassisMass}" r="${chassisLength}"/>
         </inertial>
     </link>

File: kulbu_description/urdf/macros.xacro (robot description, xacro)
@@ -41,6 +41,6 @@
         </link>
         <gazebo reference="${fb}_${lr}_wheel">
-            <mu1>1.0</mu1>
-            <mu2>1.0</mu2>
+            <mu1>${mu}</mu1>
+            <mu2>${mu}</mu2>
             <kp>1e+13</kp>
             <kd>1.0</kd>
